File: KiCAD projects/TransistorScheme/TransistorScheme.kicad_sch (KiCad schematic)
At the start: 19 parts, among them Q1 BC337, Q2 BC327-40, Q3 BC327-16, Q4 BC327-16, Q5 BC327-16, SW2 SW_SPDT

Commit message: Updated circuit and tested for room 3 using one of the circuits
Parts:
- added Rc1: 50, symbol Device:R
- added Rc2, Rc3: 100, symbol Device:R
- RV2, RV3, RV4: value 100 -> 1k
- Rb3: value 47k -> 20k
- Rb4, Rb5: value 47k -> 22k
Connections:
- net at RV4.2: now also Rc3.1; no longer D4.4 (BA)
- net at RV3.2: now also Rc1.1; no longer D4.2 (RA)
- net at RV2.2: now also Rc2.1; no longer D4.3 (GA)
- new net: D4.4 (BA), Rc3.2
- new net: D4.3 (GA), Rc2.2
- new net: D4.2 (RA), Rc1.2
Changed lines of the file:
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@@
-	(wire
-		(pts
-			(xy 172.72 104.14) (xy 186.69 104.14)
-		)
-		(stroke
-			(width 0)
-			(type default)
-		)
-	)
 	(wire
 		(pts
@@
 	(wire
 		(pts
-			(xy 186.69 123.19) (xy 196.85 123.19)
-		)
-		(stroke
-			(width 0)
-			(type default)
-		)
-	)
-	(wire
-		(pts
 			(xy 168.91 97.79) (xy 168.91 100.33)
 		)
@@
 	(wire
 		(pts
-			(xy 186.69 104.14) (xy 186.69 113.03)
+			(xy 189.23 104.14) (xy 189.23 113.03)
 		)
 		(stroke
@@
 	(wire
 		(pts
+			(xy 182.88 118.11) (xy 186.69 118.11)
+		)
+		(stroke
+			(width 0)
+			(type default)
+		)
+	)
+	(wire
+		(pts
 			(xy 160.02 104.14) (xy 160.02 102.87)
 		)
@@
 	(wire
 		(pts
-			(xy 182.88 118.11) (xy 196.85 118.11)
-		)
-		(stroke
-			(width 0)
-			(type default)
-		)
-	)
-	(wire
-		(pts
 			(xy 134.62 109.22) (xy 134.62 127)
 		)
@@
 	(wire
 		(pts
+			(xy 172.72 104.14) (xy 181.61 104.14)
+		)
+		(stroke
+			(width 0)
+			(type default)
+		)
+	)
+	(wire
+		(pts
 			(xy 134.62 109.22) (xy 139.7 109.22)
 		)
@@
 	(wire
 		(pts
-			(xy 186.69 135.89) (xy 182.88 135.89)
-		)
-		(stroke
-			(width 0)
-			(type default)
-		)
-	)
-	(wire
-		(pts
 			(xy 168.91 107.95) (xy 168.91 109.22)
 		)
@@
 	(wire
 		(pts
+			(xy 194.31 118.11) (xy 196.85 118.11)
+		)
+		(stroke
+			(width 0)
+			(type default)
+		)
+	)
+	(wire
+		(pts
 			(xy 134.62 92.71) (xy 148.59 92.71)
 		)
@@
 	(wire
 		(pts
+			(xy 182.88 135.89) (xy 186.69 135.89)
+		)
+		(stroke
+			(width 0)
+			(type default)
+		)
+	)
+	(wire
+		(pts
 			(xy 175.26 52.07) (xy 175.26 54.61)
 		)
@@
 	(wire
 		(pts
-			(xy 186.69 123.19) (xy 186.69 135.89)
+			(xy 196.85 123.19) (xy 196.85 135.89)
 		)
 		(stroke
@@
 	(wire
 		(pts
-			(xy 186.69 113.03) (xy 196.85 113.03)
+			(xy 194.31 135.89) (xy 196.85 135.89)
+		)
+		(stroke
+			(width 0)
+			(type default)
+		)
+	)
+	(wire
+		(pts
+			(xy 189.23 113.03) (xy 196.85 113.03)
 		)
 		(stroke
@@
 	(symbol
 		(lib_id "Device:R")
+		(at 190.5 135.89 90)
+		(unit 1)
+		(exclude_from_sim no)
+		(in_bom yes)
+		(on_board yes)
+		(dnp no)
+		(property "Reference" "Rc3"
+			(at 190.5 133.604 90)
+			(effects
+				(font
+					(size 1.27 1.27)
+				)
+			)
+		)
+		(property "Value" "100"
+			(at 190.5 138.176 90)
+			(effects
+				(font
+					(size 1.27 1.27)
+				)
+			)
+		)
+		(property "Footprint" ""
+			(at 190.5 137.668 90)
+			(effects
+				(font
+					(size 1.27 1.27)
+				)
+				(hide yes)
+			)
+		)
+		(property "Datasheet" "~"
+			(at 190.5 135.89 0)
+			(effects
+				(font
+					(size 1.27 1.27)
+				)
+				(hide yes)
+			)
+		)
+		(property "Description" "Resistor"
+			(at 190.5 135.89 0)
+			(effects
+				(font
+					(size 1.27 1.27)
+				)
+				(hide yes)
+			)
+		)
+		(pin "2"
+		)
+		(pin "1"
+		)
+		(instances
+			(project "TransistorScheme"
+				(path "/0063b497-d4b3-4c22-87fb-fa6b54b390f4"
+					(reference "Rc3")
+					(unit 1)
+				)
+			)
+		)
+	)
+	(symbol
+		(lib_id "Device:R")
 		(at 147.32 127 90)
 		(unit 1)
@@
 			)
 		)
-		(property "Value" "47k"
+		(property "Value" "22k"
 			(at 147.32 129.286 90)
 			(effects
@@
 			)
 		)
-		(property "Value" "47k"
+		(property "Value" "22k"
 			(at 143.51 111.506 90)
 			(effects
@@
 			)
 		)
-		(property "Value" "47k"
+		(property "Value" "20k"
 			(at 152.4 94.996 90)
 			(effects
@@
 	)
 	(symbol
+		(lib_id "Device:R")
+		(at 190.5 118.11 90)
+		(unit 1)
+		(exclude_from_sim no)
+		(in_bom yes)
+		(on_board yes)
+		(dnp no)
+		(property "Reference" "Rc2"
+			(at 190.5 115.824 90)
+			(effects
+				(font
+					(size 1.27 1.27)
+				)
+			)
+		)
+		(property "Value" "100"
+			(at 190.5 120.396 90)
+			(effects
+				(font
+					(size 1.27 1.27)
+				)
+			)
+		)
+		(property "Footprint" ""
+			(at 190.5 119.888 90)
+			(effects
+				(font
+					(size 1.27 1.27)
+				)
+				(hide yes)
+			)
+		)
+		(property "Datasheet" "~"
+			(at 190.5 118.11 0)
+			(effects
+				(font
+					(size 1.27 1.27)
+				)
+				(hide yes)
+			)
+		)
+		(property "Description" "Resistor"
+			(at 190.5 118.11 0)
+			(effects
+				(font
+					(size 1.27 1.27)
+				)
+				(hide yes)
+			)
+		)
+		(pin "2"
+		)
+		(pin "1"
+		)
+		(instances
+			(project "TransistorScheme"
+				(path "/0063b497-d4b3-4c22-87fb-fa6b54b390f4"
+					(reference "Rc2")
+					(unit 1)
+				)
+			)
+		)
+	)
+	(symbol
 		(lib_id "power:GND")
 		(at 179.07 140.97 0)
@@
 			)
 		)
-		(property "Value" "100"
+		(property "Value" "1k"
 			(at 182.88 139.954 0)
 			(effects
@@
 			)
 		)
-		(property "Value" "100"
+		(property "Value" "1k"
 			(at 172.72 108.204 0)
 			(effects
@@
 	)
 	(symbol
+		(lib_id "Device:R")
+		(at 185.42 104.14 90)
+		(unit 1)
+		(exclude_from_sim no)
+		(in_bom yes)
+		(on_board yes)
+		(dnp no)
+		(property "Reference" "Rc1"
+			(at 185.42 101.854 90)
+			(effects
+				(font
+					(size 1.27 1.27)
+				)
+			)
+		)
+		(property "Value" "50"
+			(at 185.42 106.426 90)
+			(effects
+				(font
+					(size 1.27 1.27)
+				)
+			)
+		)
+		(property "Footprint" ""
+			(at 185.42 105.918 90)
+			(effects
+				(font
+					(size 1.27 1.27)
+				)
+				(hide yes)
+			)
+		)
+		(property "Datasheet" "~"
+			(at 185.42 104.14 0)
+			(effects
+				(font
+					(size 1.27 1.27)
+				)
+				(hide yes)
+			)
+		)
+		(property "Description" "Resistor"
+			(at 185.42 104.14 0)
+			(effects
+				(font
+					(size 1.27 1.27)
+				)
+				(hide yes)
+			)
+		)
+		(pin "2"
+		)
+		(pin "1"
+		)
+		(instances
+			(project "TransistorScheme"
+				(path "/0063b497-d4b3-4c22-87fb-fa6b54b390f4"
+					(reference "Rc1")
+					(unit 1)
+				)
+			)
+		)
+	)
+	(symbol
 		(lib_id "Device:R_Potentiometer")
 		(at 179.07 118.11 0)
@@
 			)
 		)
-		(property "Value" "100"
+		(property "Value" "1k"
 			(at 182.88 122.174 0)
 			(effects
